Commit message: sensor fusion with vs controller

File: lwr_description/model/kuka_lwr.gazebo.xacro (robot description, xacro)
@@ -39,4 +39,26 @@
 			<material>Gazebo/Grey</material>
 		</gazebo>
+		<gazebo reference="${name}_palm_dummy_link">
+		</gazebo>
+        <!-- Enable the Joint Feedback -->
+<!--         <gazebo reference="${name}_6_joint">
+        <provideFeedback>true</provideFeedback>
+        </gazebo> -->
+        <!-- The ft_sensor plugin -->
+<!--         <gazebo>
+        <plugin name="ft_sensor" filename="libgazebo_ros_ft_sensor.so">
+        <updateRate>10.0</updateRate>
+        <topicName>${name}_7_link_ft_sensor_topic</topicName>
+        <jointName>${name}_6_joint</jointName>
+        <noise>
+          <type>gaussian</type> -->
+          <!-- Noise is sampled independently per pixel on each frame.
+               That pixel's noise value is added to each of its color
+               channels, which at that point lie in the range [0,1]. -->
+<!--           <mean>0.000</mean>
+          <stddev>0.000</stddev> change this to simulate noise
+        </noise>
+        </plugin>
+        </gazebo> -->
 	</xacro:macro>
 </robot>

File: lwr_description/model/kuka_lwr.urdf.xacro (robot description, xacro)
@@ -32,5 +32,5 @@
 			</inertial>
 			<visual>
-				<origin xyz="0 0 0" rpy="0 0 ${M_PI}"/>
+				<origin xyz="0 0 0" rpy="0 0 ${M_PI}"/><!-- -->
 				<geometry>
 					<mesh filename="package://lwr_description/meshes/base.STL"/>
@@ -66,5 +66,5 @@
 			<inertial>
 				<mass value="${link_mass}"/>
-				<origin rpy="0 0 0" xyz="0 -0.06 0.130"/>
+				<origin rpy="0 0 0" xyz="0 -0.06 0.130"/> <!--"-->
 				<cuboid_inertia_def length="0.12" width="0.06" height="0.260" mass="${link_mass}"/>
 			</inertial>
@@ -316,6 +316,6 @@
 			<inertial>
 				<mass value="0.2"/>
-				<origin rpy="0 0 0" xyz="0 0 0.0625"/>
-				<cuboid_inertia_def length="0.125" width="0.125" height="0.125" mass="0.2"/>
+				<origin rpy="0 0 0" xyz="0 0 0.0"/> <!--0.0625-->
+				<cuboid_inertia_def length="0.135" width="0.135" height="0.135" mass="0.2"/>
 			</inertial>
 			<visual>
@@ -353,6 +353,7 @@
 			<inertial>
 				<mass value="0.2"/>
-				<origin xyz="0 0 0"/>
-				<cuboid_inertia_def length="1" width="1" height="1" mass="0.2"/>
+				<origin xyz="0 0 -0.01" rpy="0 0 ${M_PI}" />
+				<cuboid_inertia_def length="0.02" width="0.07" height="0.07" mass="0.2"/>
+				<!--<cylinder_inertia_def radius="0.05" length="0.02" mass="0.2"/>-->
 			</inertial>
 			<visual>
@@ -370,6 +371,17 @@
 			</collision>
 		</link>
+<!--	        PALM  dummy-->
+ 		<joint name="${name}_palm_joint_dummy" type="fixed">
+				<origin xyz="0.00 +0.0 0.22" rpy="0 0 0"/>
+			<parent link="${name}_7_link" />
+			<child link="${name}_palm_dummy_link" />
+		</joint>
+		<link name="${name}_palm_dummy_link"/>
 		<xacro:kuka_lwr_gazebo name="${name}"/>
 		<xacro:kuka_lwr_transmission name="${name}"/>
+		<ros>
+		<plugin name="joint_state_estimator" filename="libjoint_state_estimator.so">
+		  </plugin>
+		</ros>
 	</xacro:macro>
 </robot>

File: single_lwr_example/single_lwr_robot/robot/single_lwr_robot.urdf.xacro (robot description, xacro)
@@ -2,17 +2,25 @@
 <robot xmlns:xacro="http://www.ros.org/wiki/xacro" name="single_lwr_robot">
 	<!-- Include all models -->
-	<xacro:include filename="$(find lwr_description)/model/kuka_lwr.urdf.xacro"/>
+   <xacro:include filename="$(find lwr_description)/model/kuka_lwr.urdf.xacro"/>
+     <xacro:include filename="$(find force_torque_sensor)/model/ft_sensor_gamma.urdf.xacro"/>
+     <xacro:include filename="$(find soft_hand_description)/model/soft_hand.urdf.xacro"/>
+  <link name="world" />
+    <joint name="world_joint" type="fixed">
+    <origin rpy="0 0 0.0" xyz="0 0 0.0"/>
+      <parent link="world"/>
+      <child link="box"/>
+   </joint>
 	<!-- and assemble your robot -->
 	<link name="box">
 		<inertial>
-			<mass value="5.0"/>
-			<origin rpy="0 0 0" xyz="0 0 0"/>
-			<inertia ixx="0.01"
-             iyy="0.01"
-             izz="0.01"
+			<mass value="50.0"/>
+			<origin rpy="0 0 0" xyz="0 0 0.5"/>
+	     <inertia ixx="8.33"
+             iyy="8.33"
+             izz="8.33"
              ixy="0" iyz="0" ixz="0"/>
 		</inertial>
 		<visual>
-			<origin xyz="0 0 0.50" rpy="0 0 0"/>
+			<origin xyz="0 0 0.5" rpy="0 0 0.0"/>
 			<geometry>
 				<box size="1.0 1.0 1.0"/>
@@ -20,5 +28,5 @@
 		</visual>
 		<collision>
-			<origin xyz="0 0 0.50" rpy="0 0 0"/>
+			<origin xyz="0 0 0.5" rpy="0 0 0.0"/>
 			<geometry>
 				<box size="1.0 1.0 1.0"/>
@@ -27,9 +35,84 @@
 	</link>
 	<gazebo reference="box">
-		<static>true</static>>
+		<static>true</static>
 	</gazebo>
 	<!-- using the models -->
 	<xacro:kuka_lwr parent="box" name="lwr">
-		<origin xyz="0 0 1" rpy="0 0 0"/>
+		<origin xyz="0 0 1.0" rpy="0 0 0"/>
 	</xacro:kuka_lwr>
+    <xacro:ft_sensor parent="lwr_7_link" name="lwr" type="gamma">
+          <origin xyz="0 0 0" rpy="0 0 0"/>
+      </xacro:ft_sensor>
+<!--      <xacro:soft_hand parent="lwr_measure" name="left_hand" left="true" withAdaptiveTransmission="true" useMimicTag="true">
+    <origin xyz="0 0 0.0025" rpy="0 0 0"/>
+  </xacro:soft_hand>-->
+ <!--     <joint name="fixed_joint" type= "fixed">
+	  <origin xyz="0 0 0.055" rpy="0 0 0"/>
+          <parent link="lwr_measure"/>
+          <child link="box_2"/>
+        </joint>-->
+	      <joint name="fixed_joint" type= "revolute">
+		<limit lower="0" upper="0" effort="0" velocity="0"/>
+	  <origin xyz="0 0 0.005" rpy="0 0 0"/>
+          <parent link="lwr_measure"/>
+          <child link="box_2"/>
+        </joint>
+	<link name="box_2">
+		<inertial>
+			<mass value="1.5"/>
+			<origin rpy="0 0 0" xyz="0 0 0.05"/>
+			<inertia ixx="0.0025"
+             iyy="0.0025"
+             izz="0.0025"
+             ixy="0.0" iyz="0.0" ixz="0.0"/>
+		</inertial>
+		<visual>
+			<origin xyz="0 0 0.05" rpy="0 0 0.0"/>
+			<geometry>
+				<box size="0.1 0.1 0.1"/>
+			</geometry>
+		</visual>
+		<collision>
+			<origin xyz="0 0 0.05" rpy="0 0 0"/>
+			<geometry>
+				<box size="0.1 0.1 0.1"/>
+			</geometry>
+		</collision>
+	</link>
+	<gazebo reference="box_2">
+		 <gravity>true</gravity>
+		 <static>true</static>
+	</gazebo>
+	<joint name="fixed_joint_2" type= "revolute">
+	  <limit lower="0" upper="0" effort="0" velocity="0"/>
+	  <origin xyz="0 0 0.1" rpy="0 0 0"/>
+          <parent link="box_2"/>
+          <child link="box_3"/>
+        </joint>
+	<link name="box_3">
+		<inertial>
+			<mass value="0.2"/>
+			<origin rpy="0 0 0" xyz="0 0 0.025"/>
+			<inertia ixx="0.000083333"
+             iyy="0.000083333"
+             izz="0.000083333"
+             ixy="0.0" iyz="0.0" ixz="0.0"/>
+		</inertial>
+		<visual>
+			<origin xyz="0 0 0.025" rpy="0 0 0"/>
+			<geometry>
+				<box size="0.05 0.05 0.05"/>
+			</geometry>
+		</visual>
+		<collision>
+			<origin xyz="0 0 0.025" rpy="0 0 0"/>
+			<geometry>
+				<box size="0.05 0.05 0.05"/>
+			</geometry>
+		</collision>
+	</link>
+	<gazebo reference="box_3">
+		 <gravity>true</gravity>
+		 <static>true</static>
+	</gazebo>
 </robot>
